Commit message: Made the suspension link rigid

File: description/joints.xacro (robot description, xacro)
@@ -1,5 +1,5 @@
 <?xml version="1.0" ?>
 <robot name="terryjr" xmlns:xacro="http://www.ros.org/wiki/xacro">
-<joint name="right_wheel_link_to_base_link_joint" type="continuous">
+<joint name="right_wheel_link_to_base_link_joint" type="fixed">
   <origin xyz="0.0 -0.192 0.307734" rpy="0 0 0"/>
   <parent link="base_link"/>
@@ -7,5 +7,5 @@
   <axis xyz="-0.0 -1.0 0.0"/>
 </joint>
-<joint name="left_wheel_link_to_base_link_joint" type="continuous">
+<joint name="left_wheel_link_to_base_link_joint" type="fixed">
   <origin xyz="0.0 0.192 0.307734" rpy="0 0 0"/>
   <parent link="base_link"/>
@@ -37,5 +37,5 @@
   <axis xyz="0.0 1.0 -0.0"/>
 </joint>
-<joint name="mid_balance_link_to_base_link_joint" type="continuous">
+<joint name="mid_balance_link_to_base_link_joint" type="fixed">
   <origin xyz="0.295 0.0 0.310934" rpy="0 0 0"/>
   <parent link="base_link"/>
@@ -43,5 +43,5 @@
   <axis xyz="1.0 0.0 -0.0"/>
 </joint>
-<joint name="right_balance_link_to_mid_balance_link_joint" type="continuous">
+<joint name="right_balance_link_to_mid_balance_link_joint" type="fixed">
   <origin xyz="0.0 -0.220009 0.0" rpy="0 0 0"/>
   <parent link="mid_balance_link"/>
@@ -49,5 +49,5 @@
   <axis xyz="1.0 0.0 -0.0"/>
 </joint>
-<joint name="left_balance_link_to_mid_balance_link_joint" type="continuous">
+<joint name="left_balance_link_to_mid_balance_link_joint" type="fixed">
   <origin xyz="0.0 0.220009 0.0" rpy="0 0 0"/>
   <parent link="mid_balance_link"/>
@@ -55,5 +55,5 @@
   <axis xyz="1.0 0.0 -0.0"/>
 </joint>
-<gazebo>
+<!-- <gazebo>
   <joint name="right_balance_link_to_right_wheel_link_joint" type="continuous">
     <pose>0.0 0.0 0.0 0 0 0</pose>
@@ -74,4 +74,4 @@
     </axis>
   </joint>
-</gazebo>
+</gazebo> -->
 </robot>

Commit message: Added a base_footprint link as per convention

File: description/joints.xacro (robot description, xacro)
@@ -1,4 +1,9 @@
 <?xml version="1.0" ?>
 <robot name="terryjr" xmlns:xacro="http://www.ros.org/wiki/xacro">
+<joint name="base_joint" type="fixed">
+  <parent link="base_footprint"/>
+  <child link="base_link"/>
+  <origin xyz="0.0 0.0 0.0" rpy="0 0 0"/>
+</joint>
 <joint name="right_wheel_link_to_base_link_joint" type="fixed">
   <origin xyz="0.0 -0.192 0.307734" rpy="0 0 0"/>

File: description/links.xacro (robot description, xacro)
@@ -1,4 +1,5 @@
 <?xml version="1.0" ?>
 <robot name="terryjr" xmlns:xacro="http://www.ros.org/wiki/xacro">
+<link name="base_footprint"/>
 <link name="base_link">
   <inertial>
